File: BitstreamEvolutionHardware/BitstreamEvolutionHardware.kicad_sch (KiCad schematic)
At the start: 0 parts

Commit message: Added Connectors Section to Sch and Linked Footprints
Parts:
- added J1, J2: PPPC101LFBN-RC, CONN10_N-RC_SUL, symbol 10PinConnector:PPPC101LFBN-RC
- added J10, J11, J12, J13, J14, J15, J16, J17, J18, J19, J20, J21, J22, J23, J24, J25, J26, J27, J28, J29, J3, J30, J31, J32, J33, J34, J4, J5, J6, J7, J8, J9: 61300211121, 61300211121, symbol 61300211121:61300211121
- added U1, U2: ADS7828, Package_SO:TSSOP-16_4.4x5mm_P0.65mm, symbol Analog_ADC:ADS7828
- added U3, U4: PPTC151LFBN-RC, PPTC151LFBN-RC, symbol PPTC151LFBN-RC:PPTC151LFBN-RC
Connections:
- new net ADC_A_Channel_0: J18.1, U2.1 (CH0)
- new net ADC_A_Channel_1: J16.1, U2.2 (CH1)
- new net ADC_A_Channel_2: J14.1, U2.3 (CH2)
- new net ADC_A_Channel_3: J12.1, U2.4 (CH3)
- new net ADC_A_Channel_4: J10.1, U2.5 (CH4)
- new net ADC_A_Channel_5: J8.1, U2.6 (CH5)
- new net ADC_A_Channel_6: J5.1, U2.7 (CH6)
- new net ADC_A_Channel_7: J6.1, U2.8 (CH7)
- new net ADC_B_Channel_0: J34.1, U1.1 (CH0)
- new net ADC_B_Channel_1: J22.1, U1.2 (CH1)
- new net ADC_B_Channel_2: J28.1, U1.3 (CH2)
- new net ADC_B_Channel_3: J33.1, U1.4 (CH3)
- new net ADC_B_Channel_4: J26.1, U1.5 (CH4)
- new net ADC_B_Channel_5: J32.1, U1.6 (CH5)
- new net ADC_B_Channel_6: J31.1, U1.7 (CH6)
- new net ADC_B_Channel_7: J30.1, U1.8 (CH7)
- new net Arduino_+3.3V: U3.P$2
- new net Arduino_+5V: U3.P$12
- new net Arduino_AREF: U3.P$3
- new net Arduino_D0: J17.1, U4.P$14
- new net Arduino_D1: J15.1, U4.P$15
- new net Arduino_D10: J21.1, U4.P$3
- new net Arduino_D11: J27.1, U4.P$2
- new net Arduino_D12: J20.1, U4.P$1
- new net Arduino_D13: J25.1, U3.P$1
- new net Arduino_D14: J24.1, U3.P$4
- new net Arduino_D15: J23.1, U3.P$5
- new net Arduino_D16: U3.P$6
- new net Arduino_D17: U3.P$7
- new net Arduino_D2: J13.1, U4.P$11
- new net Arduino_D3: J11.1, U4.P$10
- new net Arduino_D4: J9.1, U4.P$9
- new net Arduino_D5: J7.1, U4.P$8
- new net Arduino_D6: J4.1, U4.P$7
- new net Arduino_D7: J3.1, U4.P$6
- new net Arduino_D8: J29.1, U4.P$5
- new net Arduino_D9: J19.1, U4.P$4
- new net Arduino_GND: U3.P$14, U4.P$12
- new net Arduino_RESET: U4.P$13
- new net Arduino_SCL: U3.P$9
- new net Arduino_SDA: U3.P$8
- new net Arduino_VIN: U3.P$15
- new net FPGA_A_0: J1.1, J17.2, J18.2
- new net FPGA_A_1: J1.2, J15.2, J16.2
- new net FPGA_A_2: J1.3, J13.2, J14.2
- new net FPGA_A_3: J1.4, J11.2, J12.2
- new net FPGA_A_4: J1.5, J10.2, J9.2
- new net FPGA_A_5: J1.6, J7.2, J8.2
- new net FPGA_A_6: J1.7, J4.2, J5.2
- new net FPGA_A_7: J1.8, J3.2, J6.2
- new net FPGA_B_0: J2.1, J29.2, J34.2
- new net FPGA_B_1: J19.2, J2.2, J22.2
- new net FPGA_B_2: J2.3, J21.2, J28.2
- new net FPGA_B_3: J2.4, J27.2, J33.2
- new net FPGA_B_4: J2.5, J20.2, J26.2
- new net FPGA_B_5: J2.6, J25.2, J32.2
- new net FPGA_B_6: J2.7, J24.2, J31.2
- new net FPGA_B_7: J2.8, J23.2, J30.2

Commit message: Rev 0.1 Rough Draft Done
Parts:
- added C1, C2: C_Small, symbol Device:C_Small
- added J35, J36, J37, J38, J39: 61300211121, 61300211121, symbol 61300211121:61300211121
- added R1, R10, R11, R12, R2, R5, R6, R7, R8, R9: 2K, Resistor_SMD:R_0201_0603Metric, symbol Device:R_Small
- added R3, R4: 5K, Resistor_SMD:R_0201_0603Metric, symbol Device:R_Small
- added U5, U6: MAX5820MEUA+, footprints:MAX5820MEUA&plus_, symbol MAXDAC:MAX5820MEUA+
- added U7: AD9833BRMZ, SOP50P490X110-10N, symbol AD9833BRMZ:AD9833BRMZ
- added Y1: XRCGB25M000F3M04R0, footprints:OSC_XRCGB25M000F3M04R0, symbol XRCGB25M000F3M04R0:XRCGB25M000F3M04R0
- J1, J2: footprint CONN10_N-RC_SUL -> footprints:PPPC101LFBN-RC
Connections:
- net Arduino_+3.3V: now also U1.12 (A0), U1.13 (A1), U1.16 (VDD), U2.16 (VDD), C1.1, C2.1, R3.1, R4.1, U5.1 (VDD), U6.1 (VDD), U6.3 (ADD), U7.2 (VDD), Y1.1
- net Arduino_SCL: now also U1.14 (SCL), U2.14 (SCL), R12.2, R2.2, R6.2, R7.1, R9.1
- net Arduino_SDA: now also U1.15 (SDA), U2.15 (SDA), R1.2, R10.1, R11.1, R5.2, R8.1
- net ADC_REF_B: now reaches U1.10 (REF)
- net ADC_REF_B: now also J39.1
- net GND: now reaches U1.9 (GND)
- net GND: now also U2.12 (A0), U2.13 (A1), U2.9 (GND), C1.2, C2.2, J35.2, J38.2, J39.2, U5.2 (GND), U5.3 (ADD), U6.2 (GND), U7.4 (DGND), U7.9 (AGND)
- net ADC_REF_A: now reaches U2.10 (REF)
- net ADC_REF_A: now also J35.1
- new net: J36.1, U5.8 (OUTB)
- new net: J36.2, U5.7 (OUTA)
- new net: R4.2, R5.1, R6.1
- new net: R9.2, U6.4 (SCL)
- new net: R1.1, R2.1, R3.2
- new net: R10.2, U6.5 (SDA)
- new net: J37.2, U6.7 (OUTA)
- new net: J37.1, U6.8 (OUTB)
- new net: R7.2, U5.4 (SCL)
- new net: R8.2, U5.5 (SDA)
- new net: R11.2, U7.6 (SDATA)
- new net: J38.1, U7.10 (VOUT)
- new net: U7.5 (MCLK), Y1.3
- new net: R12.1, U7.7 (SCLK)
Other:
- note added: "ADC Section"
- note added: "Arduino Input"
- note added: "Connector Section"
- note added: "FPGA Input"
- note added: "Inputs for VREF Can be used to set offsets for ADC measurements"
- note added: "Waveform Generator"
- moved on the sheet: J1, J10, J11, J12, J13, J14, J15, J16, J17, J18, J19, J2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
